File: V1/PCB/WidePhoton.brd (EAGLE design)
At the start: 100 x 40 mm, 94 parts, among them IC1 PHOTON_WITH_STACKABLE_HEADERS

Commit message: Renamed files to WidePhoton Added OSH logo. Improved reverse power labels. Added diodes for battery/USB A protection. Added gitignore.
Parts:
- added D1, D2: MBRA140, SparkFun-DiscreteSemi:SMA-DIODE
- added LOGO1: OSHW-LOGOM, SparkFun-Aesthetics:OSHW-LOGO-M
Connections:
- new net N$29: D2.A, JP3.VBUS1
- new net N$31: D1.A, J1.2
- net 5V: now also D1.C, D2.C; no longer J1.2, JP3.VBUS1
Routing:
- net 5V: track 75.9 -> 43.6 mm
- net N$31: track 0.00 -> 15.1 mm, vias 0 -> 1
- net N$29: track 0.00 -> 13.3 mm
Changed lines of the file:
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@@
 <setting verticaltext="up"/>
 </settings>
-<grid distance="0.1" unitdist="mm" unit="mm" style="lines" multiple="1" display="yes" altdistance="0.05" altunitdist="mm" altunit="mm"/>
+<grid distance="0.025" unitdist="inch" unit="inch" style="lines" multiple="1" display="yes" altdistance="0.0125" altunitdist="inch" altunit="inch"/>
 <layers>
 <layer number="1" name="Top" color="4" fill="1" visible="yes" active="yes"/>
@@
 <text x="52.705" y="10.795" size="1.016" layer="26" rot="MR0">I2C
 Pull-Ups</text>
-<text x="5.08" y="27.94" size="0.8128" layer="25" font="vector">VIn</text>
-<text x="2.2225" y="27.94" size="0.8128" layer="25" font="vector">GND</text>
+<text x="4.7625" y="24.4475" size="0.8128" layer="25" font="vector">VIn</text>
+<text x="1.905" y="24.4475" size="0.8128" layer="25" font="vector">GND</text>
 <text x="64.77" y="31.75" size="0.8128" layer="26" font="vector" rot="MR270">3v3</text>
 <text x="64.77" y="24.13" size="0.8128" layer="26" font="vector" rot="MR270">GND</text>
@@
 <text x="59.69" y="32.385" size="1.4224" layer="26" font="vector" rot="MR0">3v3</text>
 <text x="8.5725" y="31.4325" size="0.8128" layer="26" font="vector" rot="MR90">3v3</text>
-<text x="49.53" y="24.765" size="1.016" layer="26" rot="MR0">+</text>
+<text x="49.53" y="13.6525" size="1.016" layer="26" rot="MR0">+</text>
 <dimension x1="4" y1="1" x2="4" y2="33" x3="-24.2" y3="17" textsize="1.016" layer="47"/>
 <dimension x1="4" y1="37" x2="4" y2="-3" x3="-27.9" y3="17" textsize="1.016" layer="47"/>
@@
 <dimension x1="4" y1="33" x2="0" y2="33" x3="2" y3="40" textsize="1.016" layer="47"/>
 <dimension x1="4" y1="33" x2="4" y2="37" x3="-3.8" y3="35" textsize="1.016" layer="47"/>
+<text x="91.7575" y="32.0675" size="0.8128" layer="25" font="vector" rot="R90">3v3</text>
+<text x="91.1225" y="32.0675" size="0.8128" layer="26" font="vector" rot="MR90">3v3</text>
+<text x="92.3925" y="-1.5875" size="0.8128" layer="26" font="vector" rot="MR0">GND</text>
+<text x="6.985" y="-0.9525" size="0.8128" layer="26" font="vector" rot="MR180">GND</text>
+<text x="3.81" y="24.4475" size="0.8128" layer="26" font="vector" rot="MR0">GND</text>
+<text x="6.6675" y="24.4475" size="0.8128" layer="26" font="vector" rot="MR0">VIn</text>
 </plain>
 <attributes>
@@
 <attribute name="VALUE" x="1.905" y="23.495" size="1.27" layer="27"/>
 </element>
+<element name="LOGO1" library="SparkFun-Aesthetics" package="OSHW-LOGO-M" value="OSHW-LOGOM" x="50.1" y="0.9"/>
+<element name="D1" library="SparkFun-DiscreteSemi" package="SMA-DIODE" value="MBRA140" x="48.895" y="30.48" rot="R180">
+<attribute name="PROD_ID" value="DIO-08053" x="48.895" y="30.48" size="1.778" layer="27" rot="R180" display="off"/>
+</element>
+<element name="D2" library="SparkFun-DiscreteSemi" package="SMA-DIODE" value="MBRA140" x="8.255" y="26.035" smashed="yes" rot="R90">
+<attribute name="PROD_ID" value="DIO-08053" x="8.255" y="26.035" size="1.778" layer="27" rot="R90" display="off"/>
+</element>
 </elements>
 <signals>
@@
 <signal name="5V">
 <contactref element="IC1" pad="1"/>
-<contactref element="JP3" pad="VBUS1"/>
 <contactref element="IC1" pad="#1"/>
 <contactref element="IC1" pad="@1"/>
 <wire x1="41.275" y1="30.48" x2="38.735" y2="30.48" width="1.016" layer="1"/>
 <wire x1="41.275" y1="30.48" x2="43.815" y2="30.48" width="1.016" layer="1"/>
-<wire x1="5.235" y1="13.645" x2="8.255" y2="13.645" width="1.016" layer="1"/>
 <wire x1="43.815" y1="30.11" x2="43.815" y2="30.48" width="0.6096" layer="1"/>
-<contactref element="J1" pad="2"/>
-<wire x1="49.165" y1="17.255" x2="48.895" y2="18.525" width="0.8128" layer="16"/>
-<wire x1="48.895" y1="18.525" x2="48.895" y2="30.48" width="0.8128" layer="16"/>
-<wire x1="48.895" y1="30.48" x2="43.815" y2="30.48" width="0.8128" layer="16"/>
-<wire x1="8.255" y1="13.645" x2="8.255" y2="26.67" width="1.016" layer="1"/>
-<wire x1="8.255" y1="26.67" x2="8.255" y2="29.21" width="1.016" layer="1"/>
 <wire x1="8.255" y1="29.21" x2="9.525" y2="30.48" width="1.016" layer="1"/>
 <wire x1="9.525" y1="30.48" x2="38.735" y2="30.48" width="1.016" layer="1"/>
 <contactref element="JP22" pad="2"/>
-<wire x1="5.715" y1="26.67" x2="8.255" y2="26.67" width="0.8128" layer="1"/>
+<contactref element="D2" pad="C"/>
+<contactref element="D1" pad="C"/>
+<wire x1="46.745" y1="30.48" x2="43.815" y2="30.48" width="0.8128" layer="1"/>
+<wire x1="8.255" y1="28.185" x2="8.255" y2="29.21" width="1.016" layer="1"/>
+<wire x1="8.255" y1="28.185" x2="6.74" y2="26.67" width="1.016" layer="1"/>
+<wire x1="6.74" y1="26.67" x2="5.715" y2="26.67" width="1.016" layer="1"/>
 </signal>
 <signal name="GND">
@@
 <wire x1="61.595" y1="25.4" x2="59.055" y2="25.4" width="0.6096" layer="16"/>
 </signal>
+<signal name="N$29">
+<contactref element="JP3" pad="VBUS1"/>
+<contactref element="D2" pad="A"/>
+<wire x1="8.255" y1="23.885" x2="8.255" y2="13.6525" width="1.016" layer="1"/>
+<wire x1="8.255" y1="13.6525" x2="5.235" y2="13.6525" width="0.8128" layer="1"/>
+<wire x1="5.235" y1="13.6525" x2="5.235" y2="13.645" width="0.8128" layer="1"/>
+</signal>
+<signal name="N$31">
+<contactref element="J1" pad="2"/>
+<contactref element="D1" pad="A"/>
+<wire x1="49.165" y1="17.255" x2="49.2125" y2="17.255" width="0.8128" layer="16"/>
+<wire x1="49.2125" y1="17.255" x2="49.2125" y2="30.48" width="0.8128" layer="16"/>
+<via x="49.2125" y="30.48" extent="1-16" drill="0.6" shape="square"/>
+<wire x1="49.2125" y1="30.48" x2="51.045" y2="30.48" width="0.8128" layer="1"/>
+</signal>
 </signals>
