File: V1/PCB/WidePhoton.sch (EAGLE design)
At the start: 94 parts, among them IC1 PHOTON_WITH_STACKABLE_HEADERS

Commit message: Renamed files to WidePhoton Added OSH logo. Improved reverse power labels. Added diodes for battery/USB A protection. Added gitignore.
Parts:
- added D1, D2: MBRA140, SparkFun-DiscreteSemi:MBRA140
- added LOGO1: OSHW-LOGOM, SparkFun-Aesthetics:OSHW-LOGOM
Connections:
- new net N$29: D2.A, JP3.VBUS
- new net N$31: D1.A, J1.+
- net 5V: now also D1.C, D2.C; no longer J1.+, JP3.VBUS
Changed lines of the file:
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@@
 <parts>
 <part name="IC1" library="Particle" deviceset="PHOTON" device="_WITH_STACKABLE_HEADERS"/>
-<part name="SUPPLY1" library="SparkFun-Aesthetics" deviceset="5V" device=""/>
 <part name="GND1" library="SparkFun-Aesthetics" deviceset="GND" device=""/>
 <part name="GND2" library="SparkFun-Aesthetics" deviceset="GND" device=""/>
@@
 <part name="SUPPLY8" library="SparkFun-Aesthetics" deviceset="5V" device=""/>
 <part name="GND8" library="SparkFun-Aesthetics" deviceset="GND" device=""/>
+<part name="LOGO1" library="SparkFun-Aesthetics" deviceset="OSHW-LOGO" device="M"/>
+<part name="D1" library="SparkFun-DiscreteSemi" deviceset="MBRA140" device=""/>
+<part name="D2" library="SparkFun-DiscreteSemi" deviceset="MBRA140" device=""/>
+<part name="SUPPLY1" library="SparkFun-Aesthetics" deviceset="5V" device=""/>
 </parts>
 <sheets>
@@
 <instances>
 <instance part="IC1" gate="G$1" x="464.82" y="-53.34"/>
-<instance part="SUPPLY1" gate="G$1" x="119.38" y="-58.42"/>
 <instance part="GND1" gate="1" x="119.38" y="-68.58"/>
 <instance part="GND2" gate="1" x="492.76" y="-40.64" rot="R90"/>
@@
 <instance part="SUPPLY8" gate="G$1" x="116.84" y="-86.36"/>
 <instance part="GND8" gate="1" x="116.84" y="-96.52"/>
+<instance part="LOGO1" gate="G$1" x="568.96" y="-172.72"/>
+<instance part="D1" gate="G$1" x="472.44" y="15.24" smashed="yes">
+<attribute name="NAME" x="474.98" y="15.7226" size="1.778" layer="95"/>
+<attribute name="VALUE" x="474.98" y="12.9286" size="1.778" layer="96"/>
+</instance>
+<instance part="D2" gate="G$1" x="119.38" y="-55.88" smashed="yes" rot="R90">
+<attribute name="NAME" x="116.3574" y="-55.88" size="1.778" layer="95" rot="R90"/>
+<attribute name="VALUE" x="124.2314" y="-58.42" size="1.778" layer="96" rot="R90"/>
+</instance>
+<instance part="SUPPLY1" gate="G$1" x="119.38" y="-48.26"/>
 </instances>
 <busses>
@@
 </segment>
 <segment>
-<pinref part="SUPPLY1" gate="G$1" pin="5V"/>
-<wire x1="119.38" y1="-58.42" x2="119.38" y2="-60.96" width="0.1524" layer="91"/>
-<wire x1="119.38" y1="-60.96" x2="132.08" y2="-60.96" width="0.1524" layer="91"/>
-<pinref part="JP3" gate="G$1" pin="VBUS"/>
-</segment>
-<segment>
-<pinref part="J1" gate="G$1" pin="+"/>
-<wire x1="464.82" y1="17.78" x2="464.82" y2="15.24" width="0.1524" layer="91"/>
-<wire x1="464.82" y1="15.24" x2="480.06" y2="15.24" width="0.1524" layer="91"/>
 <pinref part="SUPPLY7" gate="G$1" pin="5V"/>
 <wire x1="480.06" y1="15.24" x2="480.06" y2="20.32" width="0.1524" layer="91"/>
+<pinref part="D1" gate="G$1" pin="C"/>
+<wire x1="474.98" y1="15.24" x2="480.06" y2="15.24" width="0.1524" layer="91"/>
 </segment>
 <segment>
@@
 <wire x1="111.76" y1="-88.9" x2="116.84" y2="-88.9" width="0.1524" layer="91"/>
 <wire x1="116.84" y1="-88.9" x2="116.84" y2="-86.36" width="0.1524" layer="91"/>
+</segment>
+<segment>
+<pinref part="D2" gate="G$1" pin="C"/>
+<pinref part="SUPPLY1" gate="G$1" pin="5V"/>
+<wire x1="119.38" y1="-48.26" x2="119.38" y2="-53.34" width="0.1524" layer="91"/>
 </segment>
 </net>
@@
 </segment>
 </net>
+<net name="N$29" class="0">
+<segment>
+<pinref part="JP3" gate="G$1" pin="VBUS"/>
+<pinref part="D2" gate="G$1" pin="A"/>
+<wire x1="132.08" y1="-60.96" x2="119.38" y2="-60.96" width="0.1524" layer="91"/>
+<wire x1="119.38" y1="-60.96" x2="119.38" y2="-58.42" width="0.1524" layer="91"/>
+</segment>
+</net>
+<net name="N$31" class="0">
+<segment>
+<pinref part="J1" gate="G$1" pin="+"/>
+<wire x1="464.82" y1="17.78" x2="464.82" y2="15.24" width="0.1524" layer="91"/>
+<pinref part="D1" gate="G$1" pin="A"/>
+<wire x1="464.82" y1="15.24" x2="469.9" y2="15.24" width="0.1524" layer="91"/>
+</segment>
+</net>
